File: board/board.kicad_pcb (KiCad board)
At the start: 2 copper layers, 21 x 13 mm, 1 part

Commit message: schemetic finished
Parts:
- added C2: 10uF, Capacitor_SMD:C_0603_1608Metric, B.Cu at (148.0, 93.3)
- added C3: 100pF, Capacitor_SMD:C_0402_1005Metric, F.Cu at (147.8, 90.7)
- added C4: 1uF, Capacitor_SMD:C_0603_1608Metric, F.Cu at (147.7, 100.0)
- added C5: 10uF, Capacitor_SMD:C_0603_1608Metric, F.Cu at (149.2, 100.0)
- added C6: 10uF, Capacitor_SMD:C_0603_1608Metric, F.Cu at (154.9, 98.4)
- added C7: 10uF, Capacitor_SMD:C_0603_1608Metric, F.Cu at (154.9, 101.4)
- added C8: 1uF, Capacitor_SMD:C_0603_1608Metric, F.Cu at (152.7, 97.8)
- added J1: 010_UART, on_edge:on_edge_2x05_host, F.Cu at (161.0, 96.5)
- added J2: USB4105-GF-A, b051:GCT_USB4105-GF-A, F.Cu at (141.3, 96.4)
- added Q2: NXV55UN, Package_TO_SOT_SMD:SOT-23, F.Cu at (153.7, 91.8)
- added Q4: NXV55UN, Package_TO_SOT_SMD:SOT-23, F.Cu at (153.7, 95.2)
- added R1: 47.5k, Resistor_SMD:R_0603_1608Metric, B.Cu at (151.0, 91.6)
- added R10: 0R, Resistor_SMD:R_0603_1608Metric, F.Cu at (150.2, 92.3)
- added R2: 22.1k, Resistor_SMD:R_0603_1608Metric, B.Cu at (149.5, 91.6)
- added R3: 1k, Resistor_SMD:R_0603_1608Metric, B.Cu at (147.6, 97.7)
- added R4: 5.1k, Resistor_SMD:R_0402_1005Metric, F.Cu at (148.2, 94.3)
- added R5: 5.1k, Resistor_SMD:R_0402_1005Metric, F.Cu at (148.2, 98.0)
- added R6: 10k, Resistor_SMD:R_0603_1608Metric, B.Cu at (155.2, 91.6)
- added R9: 0R, Resistor_SMD:R_0603_1608Metric, F.Cu at (150.2, 90.8)
- added U1: CP2102N-Axx-xQFN28, Package_DFN_QFN:QFN-28-1EP_5x5mm_P0.5mm_EP3.35x3.35mm, B.Cu at (151.9, 96.2)
- added U2: LD39200PU33R, b121:SON95P300X300X100-7N, F.Cu at (152.0, 100.3)
- moved LOGO1 32.8 mm to (156.9, 131.1)
Routing:
- net GND: track 0.00 -> 52.1 mm, vias 0 -> 5
- net +5V: track 0.00 -> 32.7 mm, vias 0 -> 2
- net +3.3V: track 0.00 -> 30.5 mm, vias 0 -> 2
- net Net-(C3-Pad1): track 0.00 -> 19.5 mm
- net /cp2102/RTS: track 0.00 -> 18.2 mm, vias 0 -> 1
- net /cp2102/DRT: track 0.00 -> 14.5 mm, vias 0 -> 1
- net /cp2102/~{reset}: track 0.00 -> 13.9 mm
- net /cp2102/USRT_TX: track 0.00 -> 11.8 mm, vias 0 -> 1
- net /cp2102/UART_RX: track 0.00 -> 9.07 mm, vias 0 -> 1
- net /cp2102/USB_DM: track 0.00 -> 6.59 mm, vias 0 -> 1
- net /cp2102/USB_DP: track 0.00 -> 5.90 mm, vias 0 -> 1
- net Net-(J1-~{RESET}): track 0.00 -> 4.54 mm, vias 0 -> 1
- net Net-(J1-CS/EN): track 0.00 -> 4.26 mm, vias 0 -> 1
- net Net-(Q4-G): track 0.00 -> 4.16 mm
- net Net-(U1-~{SUSPEND}): track 0.00 -> 3.94 mm
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Other:
- outline, holes or cut-outs redrawn
