File: board/board.kicad_pcb (KiCad board)
At the start: 2 copper layers, 21 x 13 mm, 22 parts, among them J1 010_UART, J2 USB4105-GF-A, Q2 NXV55UN, Q4 NXV55UN, U1 CP2102N-Axx-xQFN28, U2 LD39200PU33R

Commit message: layout finished
Parts:
- added C1: 1uF, Capacitor_SMD:C_0603_1608Metric, F.Cu at (149.7, 95.2)
- LOGO1: moved to B.Cu
- moved LOGO1 37.5 mm to (143.5, 96.1), turned to 180 degrees
- moved R4 0.38 mm to (148.1, 94.0)
- moved C4 0.05 mm to (147.6, 100.0)
- moved C5 0.05 mm to (149.1, 100.0)
Connections:
- net /cp2102/DRT renamed /cp2102/DTR
Routing:
- net Net-(U1-VBUS): track 2.76 -> 4.79 mm, vias 0 -> 1
- net /cp2102/DTR: track 14.5 -> 15.1 mm
Other:
- board text added: "osf.010"
- board text added: "osf.c004.v1.0"
