File: board/usb-c.kicad_sch (KiCad schematic)
At the start: 4 parts, among them J2 USB4105-GF-A

Commit message: schemetic finished
Parts:
- removed C3: 100pF, Capacitor_SMD:C_0402_1005Metric, symbol Device:C_Small
- removed R7, R8: 5.1k, Resistor_SMD:R_0402_1005Metric, symbol Device:R_Small
- added C1: 100pF, Capacitor_SMD:C_0402_1005Metric, symbol Device:C_Small
- added R3, R4: 5.1k, Resistor_SMD:R_0402_1005Metric, symbol Device:R_Small
Connections:
- net GND: now also C1.2, R3.2, R4.2
- net at J2.A5 (CC1): now also R3.1
- net at J2.B5 (CC2): now also R4.1
- net at J2.G1 (SCHIELD), J2.G2 (SCHIELD), J2.G3 (SCHIELD)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: now also C1.1
