File: board/board.kicad_sch (KiCad schematic)
At the start: 2 parts, among them J1 010_UART

Commit message: schemetic finished
Parts:
- added Q1, Q3: NXV55UN, Package_TO_SOT_SMD:SOT-23, symbol board-rescue:Q_NMOS_GSD-parts
- added R4, R5: 0R, Resistor_SMD:R_0603_1608Metric, symbol Device:R_Small
- J1: footprint (none) -> on_edge:on_edge_2x05_host
Connections:
- net +5V: now also J1.10 (5V)
- net GND: now also J1.1 (GND)
- net cp2102/UART_CS: no longer names the net of J1.6 (CS/EN)
- net cp2102/UART_CS: now also Q3.3 (D)
- net cp2102/~{UART_reset}: no longer names the net of J1.7 (~{RESET})
- net cp2102/~{UART_reset}: now also Q1.3 (D)
- new net: Q3.1 (G), R4.2
- new net: Q1.1 (G), R5.2
- new net cp2102/DRT: Q3.2 (S), R5.1
- new net cp2102/RTS: Q1.2 (S), R4.1
- no-connect marks 2 -> 3
Other:
- removed sheet usb
- added sheet ldo (ldo.kicad_sch)
- added sheet usb-c (usb-c.kicad_sch)
- sheet cp2102 ports: added DRT, RTS; removed UART_CS, ~{UART_reset}
- moved on the sheet: J1

Commit message: layout finished
Connections:
- net cp2102/DRT renamed cp2102/DTR
Other:
- sheet cp2102 ports: added DTR; removed DRT
Changed lines of the file:
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@@
       (effects (font (size 1.27 1.27)) (justify right))
     )
-    (pin "DRT" input (at 195.58 126.365 0)
+    (pin "DTR" input (at 195.58 126.365 0)
       (effects (font (size 1.27 1.27)) (justify right))
     )
