File: board/cp2102.kicad_sch (KiCad schematic)
At the start: 11 parts, among them Q1 AO3400A, Q3 AO3400A, U1 CP2102N-Axx-xQFN28

Commit message: schemetic finished
Parts:
- removed Q1, Q3: AO3400A, parts:SOT-23, symbol board-rescue:Q_NMOS_GSD-parts
- removed R4, R5: 0R, Resistor_SMD:R_0603_1608Metric, symbol Device:R_Small
- C2: footprint (none) -> Capacitor_SMD:C_0603_1608Metric
- R1, R2, R3, R6: footprint (none) -> Resistor_SMD:R_0603_1608Metric
Connections:
- net RTS: now reaches U1.24 (~{RTS})
- net DRT: now reaches U1.28 (~{DTR})

Commit message: layout finished
Parts:
- C1: footprint (none) -> Capacitor_SMD:C_0603_1608Metric
Connections:
- net DRT renamed DTR
Changed lines of the file:
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@@
     (effects (font (size 1.27 1.27)) (justify right))
   )
-  (hierarchical_label "DRT" (shape input) (at 175.895 81.915 0) (fields_autoplaced)
+  (hierarchical_label "DTR" (shape input) (at 175.895 81.915 0) (fields_autoplaced)
     (effects (font (size 1.27 1.27)) (justify left))
   )
@@
       (effects (font (size 1.27 1.27)) (justify left))
     )
-    (property "Footprint" "" (at 125.73 86.36 0)
+    (property "Footprint" "Capacitor_SMD:C_0603_1608Metric" (at 125.73 86.36 0)
       (effects (font (size 1.27 1.27)) hide)
     )
